File: kicad/mems_mic_board.kicad_pcb (KiCad board)
At the start: 2 copper layers, 10 parts, among them J1 Conn_01x02_Male, J2 Conn_01x03_Male, J3 Conn_01x06_Male, J4 Conn_01x02_Male, J5 Conn_01x04_Male, J6 Conn_01x08_Male, J7 Conn_01x08_Male, U1 tactile_sw, U2 mems_mic, U3 mems_mic

Commit message: update
Parts:
- removed J5: Conn_01x04_Male, mcu:Pin Header 4P
- J1: value Conn_01x02_Male -> Conn_01x06_Male; footprint mcu:Pin Header 2P -> mcu:Pin Header 6P
- J2: value Conn_01x03_Male -> Conn_01x01_Male; footprint mcu:Pin_Header_3P -> mcu:Pin_header_1P
- J4: value Conn_01x02_Male -> Conn_01x06_Female; footprint mcu:Pin Header 2P -> mcu:Pin Header 6P
- moved J4 50.0 mm to (141.0, 90.2)
- moved J2 24.1 mm to (119.4, 135.9), turned to 0 degrees
- moved U2 7.62 mm to (125.7, 91.4)
- moved U3 7.62 mm to (125.7, 132.1)
- moved J1 5.08 mm to (111.8, 109.2)
- moved U1 1.27 mm to (110.5, 94.0)
Connections:
- J2 pad 1: GND -> Net-(J2-Pad1)
- J4 pad 1: Net-(J4-Pad1) -> GND
- J7 pad 7: Net-(J5-Pad4) -> Net-(J4-Pad4)
- J7 pad 8: Net-(J5-Pad3) -> Net-(J4-Pad5)
- U2 pad 4: Net-(J4-Pad2) -> Net-(J2-Pad1)
- U3 pad 4: Net-(J4-Pad2) -> Net-(J2-Pad1)
Routing:
- net +3V3: track 167.6 -> 66.0 mm, vias 0 -> 6
- net Net-(J4-Pad1): track 58.4 -> 0.00 mm, vias 6 -> 0
- net Net-(J4-Pad2): track 55.9 -> 0.00 mm, vias 2 -> 0
- net Net-(J4-Pad5): track 0.00 -> 53.3 mm
- net Net-(J4-Pad4): track 0.00 -> 53.3 mm, vias 0 -> 2
- net Net-(J2-Pad1): track 0.00 -> 53.3 mm, vias 0 -> 4
- net Net-(J1-Pad3): track 0.00 -> 45.7 mm, vias 0 -> 2
- net GND: track 124.5 -> 90.2 mm, vias 2 -> 0
- net Net-(J5-Pad4): track 20.3 -> 0.00 mm, vias 2 -> 0
- net Net-(J5-Pad3): track 15.2 -> 0.00 mm, vias 2 -> 0
- net Net-(J1-Pad1): track 22.9 -> 21.6 mm, vias 2 -> 0
- net Net-(J6-Pad7): vias 2 -> 6

Commit message: update
Parts:
- moved J4 2.54 mm to (141.0, 87.6)
Routing:
- net Net-(J4-Pad5): track 53.3 -> 55.9 mm
- net Net-(J4-Pad4): track 53.3 -> 55.9 mm
- net Net-(J1-Pad3): track 45.7 -> 48.3 mm
- net GND: track 90.2 -> 92.7 mm
Changed lines of the file:
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@@
     (links 16)
     (no_connects 0)
-    (area 0 0 0 0)
+    (area 105.084999 84.115 158.555 139.505)
     (thickness 1.6)
     (drawings 4)
@@
       (outputformat 1)
       (mirror false)
-      (drillshape 1)
+      (drillshape 0)
       (scaleselection 1)
       (outputdirectory ""))
@@
   )
   (module "mcu:Pin Header 6P" (layer F.Cu)
-    (at 140.97 90.17)
+    (at 140.97 87.63)
     (fp_text reference J4 (at 0 2.54) (layer F.SilkS)
       (effects (font (size 1 1) (thickness 0.15)))
@@
   (via (at 127 105.41) (size 0.6) (drill 0.4) (layers F.Cu B.Cu) (net 2))
   (segment (start 111.76 107.95) (end 114.3 107.95) (width 0.25) (layer B.Cu) (net 3))
-  (segment (start 139.7 107.95) (end 139.7 90.17) (width 0.25) (layer B.Cu) (net 3) (status 20))
+  (segment (start 139.7 107.95) (end 139.7 87.63) (width 0.25) (layer B.Cu) (net 3) (status 20))
   (segment (start 121.92 107.95) (end 139.7 107.95) (width 0.25) (layer B.Cu) (net 3))
   (via (at 121.92 107.95) (size 0.6) (drill 0.4) (layers F.Cu B.Cu) (net 3))
@@
   (segment (start 121.92 130.81) (end 121.92 128.27) (width 0.25) (layer B.Cu) (net 4))
   (segment (start 111.76 110.49) (end 116.84 110.49) (width 0.25) (layer B.Cu) (net 4))
-  (segment (start 134.62 90.17) (end 134.62 93.98) (width 0.25) (layer B.Cu) (net 4) (status 10))
+  (segment (start 134.62 87.63) (end 134.62 93.98) (width 0.25) (layer B.Cu) (net 4) (status 10))
   (segment (start 134.62 93.98) (end 134.62 100.33) (width 0.25) (layer B.Cu) (net 4))
   (segment (start 134.62 100.33) (end 129.54 100.33) (width 0.25) (layer B.Cu) (net 4))
@@
   (segment (start 119.38 135.89) (end 121.92 135.89) (width 0.25) (layer B.Cu) (net 7))
   (segment (start 154.94 130.81) (end 149.86 130.81) (width 0.25) (layer B.Cu) (net 15))
-  (segment (start 142.24 130.81) (end 142.24 90.17) (width 0.25) (layer B.Cu) (net 15) (status 20))
+  (segment (start 142.24 130.81) (end 142.24 87.63) (width 0.25) (layer B.Cu) (net 15) (status 20))
   (via (at 142.24 130.81) (size 0.6) (drill 0.4) (layers F.Cu B.Cu) (net 15))
   (segment (start 149.86 130.81) (end 142.24 130.81) (width 0.25) (layer F.Cu) (net 15))
   (via (at 149.86 130.81) (size 0.6) (drill 0.4) (layers F.Cu B.Cu) (net 15))
-  (segment (start 144.78 90.17) (end 144.78 133.35) (width 0.25) (layer B.Cu) (net 16) (status 10))
+  (segment (start 144.78 87.63) (end 144.78 133.35) (width 0.25) (layer B.Cu) (net 16) (status 10))
   (segment (start 144.78 133.35) (end 154.94 133.35) (width 0.25) (layer B.Cu) (net 16) (status 20))
   (segment (start 129.54 95.25) (end 132.08 95.25) (width 0.25) (layer B.Cu) (net 24))

Commit message: update
Parts:
- removed J4: Conn_01x06_Female, mcu:Pin Header 6P
- moved U3 12.7 mm to (133.3, 121.9)
- moved U2 12.7 mm to (133.3, 101.6)
- moved J2 10.2 mm to (129.5, 135.9)
- moved U1 9.25 mm to (119.4, 91.4)
Routing:
- net Net-(J4-Pad5): track 55.9 -> 0.00 mm
- net Net-(J4-Pad4): track 55.9 -> 0.00 mm, vias 2 -> 0
- net Net-(J1-Pad3): track 48.3 -> 0.00 mm, vias 2 -> 0
- net GND: track 92.7 -> 58.4 mm, vias 0 -> 2
- net Net-(J6-Pad7): track 73.7 -> 40.6 mm, vias 6 -> 0
- net Net-(J2-Pad1): track 53.3 -> 38.1 mm, vias 4 -> 0
- net +3V3: track 66.0 -> 55.9 mm, vias 6 -> 2
- net Net-(J1-Pad1): track 21.6 -> 20.3 mm

Commit message: update pattern
Parts:
- removed J6, J7: Conn_01x08_Male, mcu:Pin Header 8P
- added J4: Conn_01x10_Male, mcu:Pin Header 10P, F.Cu at (154.9, 100.3)
- added J5: Conn_01x08_Male, mcu:Pin Header 8P, F.Cu at (154.9, 125.7)
- J1: value Conn_01x06_Male -> Conn_01x08_Male; footprint mcu:Pin Header 6P -> mcu:Pin Header 8P
- J2: value Conn_01x01_Male -> Conn_01x06_Male; footprint mcu:Pin_header_1P -> mcu:Pin Header 6P
- J3: value Conn_01x06_Male -> Conn_01x01_Male; footprint mcu:Pin Header 6P -> mcu:Pin_header_1P
- moved J3 20.5 mm to (129.5, 137.2), turned to 0 degrees
- moved J2 19.3 mm to (111.8, 128.3), turned to 270 degrees
- moved U1 1.80 mm to (118.1, 90.2)
- moved U2 1.27 mm to (133.3, 102.9)
- moved J1 1.27 mm to (111.8, 108.0)
- moved U3 1.27 mm to (133.3, 123.2)
Connections:
- J1 pad 2: +3V3 -> Net-(J1-Pad2)
- J1 pad 4: GND -> +3V3
- J1 pad 6: Net-(J1-Pad6) -> GND
- U1 pad 1: GND -> Net-(U1-Pad1)
- U1 pad 2: Net-(U1-Pad2) -> GND
- U1 pad 3: Net-(J1-Pad1) -> Net-(U1-Pad3)
- U1 pad 4: Net-(U1-Pad4) -> Net-(J1-Pad3)
- U2 pad 4: Net-(J2-Pad1) -> Net-(J3-Pad1)
- U3 pad 4: Net-(J2-Pad1) -> Net-(J3-Pad1)
Routing:
- net Net-(J3-Pad1): track 0.00 -> 38.1 mm
- net Net-(J2-Pad1): track 38.1 -> 0.00 mm
- net Net-(J1-Pad1): track 20.3 -> 0.00 mm
- net +3V3: track 55.9 -> 71.1 mm
- net Net-(J1-Pad3): track 0.00 -> 14.0 mm
- net GND: track 58.4 -> 55.9 mm, vias 2 -> 0
- net Net-(J4-Pad9): track 40.6 -> 43.2 mm

Commit message: update
Parts:
- added J6: Conn_01x04_Female, mcu:pin-socket-4p, F.Cu at (135.9, 137.2)
Connections:
- J1 pad 5: Net-(J1-Pad5) -> /5V
- J4 pad 1: Net-(J4-Pad1) -> /SCL
- J4 pad 2: Net-(J4-Pad2) -> /SDA
Routing:
- net /SCL: track 0.00 -> 68.6 mm, vias 0 -> 3
- net /SDA: track 0.00 -> 63.5 mm, vias 0 -> 3
- net /5V: track 0.00 -> 48.3 mm, vias 0 -> 3
- net GND: track 55.9 -> 91.4 mm, vias 0 -> 3

Commit message: update
Parts:
- removed U2: mems_mic, mcu:MEMS_mic
- J6: value Conn_01x04_Female -> Conn_01x06_Female; footprint mcu:pin-socket-4p -> mcu:Pin_Socket_6P
- moved U3 17.8 mm to (134.6, 105.4)
- moved J3 17.6 mm to (120.7, 121.9)
- moved J6 7.73 mm to (134.6, 129.5)
- moved U1 2.54 mm to (120.7, 90.2)
- moved J1 2.54 mm to (114.3, 108.0)
- moved J2 2.54 mm to (114.3, 128.3)
Connections:
- J1 pad 5: /5V -> U5V
- J4 pad 1: /SCL -> Net-(J4-Pad1)
- J4 pad 2: /SDA -> Net-(J4-Pad2)
- J6 pad 1: /5V -> Net-(J6-Pad1)
- J6 pad 2: /SCL -> Net-(J5-Pad6)
- J6 pad 3: /SDA -> Net-(J4-Pad10)
- J6 pad 4: GND -> U5V
Routing:
- net /SCL: track 68.6 -> 0.00 mm, vias 3 -> 0
- net /SDA: track 63.5 -> 0.00 mm, vias 3 -> 0
- net /5V: track 48.3 -> 0.00 mm, vias 3 -> 0
- net Net-(J4-Pad10): track 0.00 -> 44.5 mm
- net U5V: track 0.00 -> 41.9 mm, vias 0 -> 2
- net +3V3: track 71.1 -> 34.3 mm
- net Net-(J5-Pad6): track 0.00 -> 34.3 mm
- net Net-(J4-Pad9): track 43.2 -> 16.5 mm
- net Net-(J3-Pad1): track 38.1 -> 22.9 mm
- net GND: track 91.4 -> 77.5 mm, vias 3 -> 0
